Commit message: Isaac Sim: port mundo+dron+sensores+ArUcos 3D+HUD+multicamara; rodillos cilindricos (serpenteo -40%)
Port del sim Gazebo a Isaac Sim 4.5, integrado en scene_mecanum.py con flags componibles
(--world laberinto, --lidar, --imu, --camera, --aruco, --drone, --cameras/--rec_cams, --perf + knobs de
fisica del serpenteo). La escena por defecto (Kalman/gridmap) queda intacta.

Modulos nuevos:
- world_loader.py: laberinto Gazebo en Isaac via STL->USD (asset_converter) + colision de malla 'none' +
  colores planos = Gazebo + rotacion Rx90*Rz90 + auto-centrado. (NO por URDF: dejaba convexHull.)
- drone.py: dron Tello KINEMATICO que obedece /drone1/cmd_vel; camara nadir /uav/camera/image+info;
  /drone1/odom; takeoff/land.
- aruco3d.py: ArUcos 3D reales (tabla blanca 4mm + celdas negras extruidas +0.6mm); cubo objetivo + ID4 techo.
- sensors.py: IMU /imu/data_raw + camara RGB-D /cam_1/* via OmniGraph (anadir nodos al /ActionGraph existente).
- cameras.py: rig multicamara (scene/chase/wheel) + grabacion replicator + viewports + presets de resolucion.
- perf_hud.py: FPS/RTF/GPU/mem en consola + /isaac/perf + overlay de stats GUI.
- serpenteo_sweep.py: barrido de knobs + regen parametrico de rodillos (sphere|cylinder|capsule).
- tello_action_shim.py + launch_ros_stack.sh: stack ROS (stitching/nav) corriendo en host (dominio 30)
  contra Isaac; shim TelloAction->topics Empty del dron.

Serpenteo: rodillos CILINDRICOS por defecto en jetauto_mecanum.urdf -> residual 1.6cm->1.0cm (-40%) y
tracking RMS -52%. (Invariante a friccion/#rodillos/controlador/solver-iters; el contacto de linea del barril
es lo que ayuda y es lo mas sim-to-real.)

Docs: INTEGRATION_GUIDE.md + PORT_NIGHTLY_REPORT.md.

File: isaac/assets/jetauto_mecanum.urdf (robot description, URDF)
Before this commit: robot jetauto, 62 links, 61 joints
Links:
- link back_left_roller_0_link: geometry collision cylinder length=0.018 radius=0.0096
- link back_left_roller_10_link: geometry collision cylinder length=0.018 radius=0.0096
- link back_left_roller_11_link: geometry collision cylinder length=0.018 radius=0.0096
- link back_left_roller_1_link: geometry collision cylinder length=0.018 radius=0.0096
- link back_left_roller_2_link: geometry collision cylinder length=0.018 radius=0.0096
- link back_left_roller_3_link: geometry collision cylinder length=0.018 radius=0.0096
- link back_left_roller_4_link: geometry collision cylinder length=0.018 radius=0.0096
- link back_left_roller_5_link: geometry collision cylinder length=0.018 radius=0.0096
- link back_left_roller_6_link: geometry collision cylinder length=0.018 radius=0.0096
- link back_left_roller_7_link: geometry collision cylinder length=0.018 radius=0.0096
- link back_left_roller_8_link: geometry collision cylinder length=0.018 radius=0.0096
- link back_left_roller_9_link: geometry collision cylinder length=0.018 radius=0.0096
- link back_left_wheel_link: geometry visual mesh filename=file:///home/opyntorr/agv_uav_project_jetauto/src/mi_proyec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
- link back_right_roller_0_link: geometry collision cylinder length=0.018 radius=0.0096
- link back_right_roller_10_link: geometry collision cylinder length=0.018 radius=0.0096
- link back_right_roller_11_link: geometry collision cylinder length=0.018 radius=0.0096
- link back_right_roller_1_link: geometry collision cylinder length=0.018 radius=0.0096
- link back_right_roller_2_link: geometry collision cylinder length=0.018 radius=0.0096
- link back_right_roller_3_link: geometry collision cylinder length=0.018 radius=0.0096
- link back_right_roller_4_link: geometry collision cylinder length=0.018 radius=0.0096
- link back_right_roller_5_link: geometry collision cylinder length=0.018 radius=0.0096
- link back_right_roller_6_link: geometry collision cylinder length=0.018 radius=0.0096
- link back_right_roller_7_link: geometry collision cylinder length=0.018 radius=0.0096
- link back_right_roller_8_link: geometry collision cylinder length=0.018 radius=0.0096
- link back_right_roller_9_link: geometry collision cylinder length=0.018 radius=0.0096
- link back_right_wheel_link: geometry visual mesh filename=file:///home/opyntorr/agv_uav_project_jetauto/src/mi_proyec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
- link back_shell_link: geometry visual mesh filename=file:///home/opyntorr/agv_uav_project_jetauto/src/mi_proyec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
- link base_link: geometry collision box size=0.297 0.145 0.11255; visual mesh filename=file:///home/opyntorr/agv_uav_project_jetauto/src/mi_proyec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
- link cam_1_link: geometry visual mesh filename=file:///home/opyntorr/agv_uav_project_jetauto/src/mi_proyec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
- link front_left_roller_0_link: geometry collision cylinder length=0.018 radius=0.0096
- link front_left_roller_10_link: geometry collision cylinder length=0.018 radius=0.0096
- link front_left_roller_11_link: geometry collision cylinder length=0.018 radius=0.0096
- link front_left_roller_1_link: geometry collision cylinder length=0.018 radius=0.0096
- link front_left_roller_2_link: geometry collision cylinder length=0.018 radius=0.0096
- link front_left_roller_3_link: geometry collision cylinder length=0.018 radius=0.0096
- link front_left_roller_4_link: geometry collision cylinder length=0.018 radius=0.0096
- link front_left_roller_5_link: geometry collision cylinder length=0.018 radius=0.0096
- link front_left_roller_6_link: geometry collision cylinder length=0.018 radius=0.0096
- link front_left_roller_7_link: geometry collision cylinder length=0.018 radius=0.0096
- link front_left_roller_8_link: geometry collision cylinder length=0.018 radius=0.0096
- link front_left_roller_9_link: geometry collision cylinder length=0.018 radius=0.0096
- link front_left_wheel_link: geometry visual mesh filename=file:///home/opyntorr/agv_uav_project_jetauto/src/mi_proyec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
- link front_right_roller_0_link: geometry collision cylinder length=0.018 radius=0.0096
- link front_right_roller_10_link: geometry collision cylinder length=0.018 radius=0.0096
- link front_right_roller_11_link: geometry collision cylinder length=0.018 radius=0.0096
- link front_right_roller_1_link: geometry collision cylinder length=0.018 radius=0.0096
- link front_right_roller_2_link: geometry collision cylinder length=0.018 radius=0.0096
- link front_right_roller_3_link: geometry collision cylinder length=0.018 radius=0.0096
- link front_right_roller_4_link: geometry collision cylinder length=0.018 radius=0.0096
- link front_right_roller_5_link: geometry collision cylinder length=0.018 radius=0.0096
- link front_right_roller_6_link: geometry collision cylinder length=0.018 radius=0.0096
- link front_right_roller_7_link: geometry collision cylinder length=0.018 radius=0.0096
- link front_right_roller_8_link: geometry collision cylinder length=0.018 radius=0.0096
- link front_right_roller_9_link: geometry collision cylinder length=0.018 radius=0.0096
- link front_right_wheel_link: geometry visual mesh filename=file:///home/opyntorr/agv_uav_project_jetauto/src/mi_proyec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
- link lidar_link: geometry visual mesh filename=file:///home/opyntorr/agv_uav_project_jetauto/src/mi_proyec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
- link mic_link: geometry visual mesh filename=file:///home/opyntorr/agv_uav_project_jetauto/src/mi_proyec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
- link speaker_link: geometry visual mesh filename=file:///home/opyntorr/agv_uav_project_jetauto/src/mi_proyec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

Commit message: Snapshot Vilchis: stack Isaac + mision dron, paquetes y assets
Isaac:
- Ajustes en scene_mecanum, world_loader, jetauto_materials, aruco3d,
  perf_hud, launch_ros_stack, isaac_env y URDF mecanum
- Probes top-down/cam (auxiliares)

mi_proyecto_sim:
- Pipeline de mision/stitching (mision/: stitch_sift, solve_global,
  refine_window, blend_vote, tape_snap, place_pose, io_utils, debug)
- Nodos nuevos: amcl_localizer, planificador_astar, generador_mapa,
  slam_occupancy_grid, filtro_lidar, odom_noise_filter, detector_aruco,
  nav_goal_bridge, control_trayectoria, Mcnamu_driver_PID(_sim), etc.
- Launches (mapeo/nav/mision/control real y sim) y configs (amcl,
  cartographer, controllers_pid, mapper_params, xbox_mecanum)
- URDF/meshes jetauto, modelos (arucos, dron, laberinto_real, tello)
- Mapas y arucos.yaml

Vendor / extras:
- yahboom_* (base, description, msgs, rosmaster, ydlidar)
- rf2o_laser_odometry (aplanado a archivos normales)
- demo_tello_sim, tello_control_pos, jetauto_rviz, jetauto_teleop
- mi_proyecto_sim_original_gazebo (referencia Gazebo)
- Integration2_FiltroKalman.zip, Integration3_MapaOcupacion.zip

gitignore:
- Excluye core dumps (core, core.*) y mision_output/ (salidas
  regenerables por corrida)

File: isaac/assets/jetauto_mecanum.urdf (robot description, URDF)
Before this commit: robot jetauto, 62 links, 61 joints
Links:
- added link aruco_black_link; visual mesh filename=file:///home/opyntorr/agv_uav_project_jetauto/src/mi_proyec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 scale=0.001 0.001 0.001
- added link aruco_link, mass 0.03; visual mesh filename=file:///home/opyntorr/agv_uav_project_jetauto/src/mi_proyec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 scale=0.001 0.001 0.001
- added link lidar_a1_frame
- added link ms200_link, mass 0.05; collision box size=0.038 0.038 0.030; visual mesh filename=file:///home/opyntorr/agv_uav_project_jetauto/src/mi_proyec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 scale=0.001 0.001 0.001
- added link screen_link, mass 0.247926; visual mesh filename=file:///home/opyntorr/agv_uav_project_jetauto/src/mi_proyec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
- added link support_link, mass 0.20; collision box size=0.150 0.185 0.173; visual mesh filename=file:///home/opyntorr/agv_uav_project_jetauto/src/mi_proyec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 scale=0.001 0.001 0.001
- link back_left_roller_0_link: geometry collision capsule length=0.018 radius=0.0096
- link back_left_roller_10_link: geometry collision capsule length=0.018 radius=0.0096
- link back_left_roller_11_link: geometry collision capsule length=0.018 radius=0.0096
- link back_left_roller_1_link: geometry collision capsule length=0.018 radius=0.0096
- link back_left_roller_2_link: geometry collision capsule length=0.018 radius=0.0096
- link back_left_roller_3_link: geometry collision capsule length=0.018 radius=0.0096
- link back_left_roller_4_link: geometry collision capsule length=0.018 radius=0.0096
- link back_left_roller_5_link: geometry collision capsule length=0.018 radius=0.0096
- link back_left_roller_6_link: geometry collision capsule length=0.018 radius=0.0096
- link back_left_roller_7_link: geometry collision capsule length=0.018 radius=0.0096
- link back_left_roller_8_link: geometry collision capsule length=0.018 radius=0.0096
- link back_left_roller_9_link: geometry collision capsule length=0.018 radius=0.0096
- link back_right_roller_0_link: geometry collision capsule length=0.018 radius=0.0096
- link back_right_roller_10_link: geometry collision capsule length=0.018 radius=0.0096
- link back_right_roller_11_link: geometry collision capsule length=0.018 radius=0.0096
- link back_right_roller_1_link: geometry collision capsule length=0.018 radius=0.0096
- link back_right_roller_2_link: geometry collision capsule length=0.018 radius=0.0096
- link back_right_roller_3_link: geometry collision capsule length=0.018 radius=0.0096
- link back_right_roller_4_link: geometry collision capsule length=0.018 radius=0.0096
- link back_right_roller_5_link: geometry collision capsule length=0.018 radius=0.0096
- link back_right_roller_6_link: geometry collision capsule length=0.018 radius=0.0096
- link back_right_roller_7_link: geometry collision capsule length=0.018 radius=0.0096
- link back_right_roller_8_link: geometry collision capsule length=0.018 radius=0.0096
- link back_right_roller_9_link: geometry collision capsule length=0.018 radius=0.0096
- link front_left_roller_0_link: geometry collision capsule length=0.018 radius=0.0096
- link front_left_roller_10_link: geometry collision capsule length=0.018 radius=0.0096
- link front_left_roller_11_link: geometry collision capsule length=0.018 radius=0.0096
- link front_left_roller_1_link: geometry collision capsule length=0.018 radius=0.0096
- link front_left_roller_2_link: geometry collision capsule length=0.018 radius=0.0096
- link front_left_roller_3_link: geometry collision capsule length=0.018 radius=0.0096
- link front_left_roller_4_link: geometry collision capsule length=0.018 radius=0.0096
- link front_left_roller_5_link: geometry collision capsule length=0.018 radius=0.0096
- link front_left_roller_6_link: geometry collision capsule length=0.018 radius=0.0096
- link front_left_roller_7_link: geometry collision capsule length=0.018 radius=0.0096
- link front_left_roller_8_link: geometry collision capsule length=0.018 radius=0.0096
- link front_left_roller_9_link: geometry collision capsule length=0.018 radius=0.0096
- link front_right_roller_0_link: geometry collision capsule length=0.018 radius=0.0096
- link front_right_roller_10_link: geometry collision capsule length=0.018 radius=0.0096
- link front_right_roller_11_link: geometry collision capsule length=0.018 radius=0.0096
- link front_right_roller_1_link: geometry collision capsule length=0.018 radius=0.0096
- link front_right_roller_2_link: geometry collision capsule length=0.018 radius=0.0096
- link front_right_roller_3_link: geometry collision capsule length=0.018 radius=0.0096
- link front_right_roller_4_link: geometry collision capsule length=0.018 radius=0.0096
- link front_right_roller_5_link: geometry collision capsule length=0.018 radius=0.0096
- link front_right_roller_6_link: geometry collision capsule length=0.018 radius=0.0096
- link front_right_roller_7_link: geometry collision capsule length=0.018 radius=0.0096
- link front_right_roller_8_link: geometry collision capsule length=0.018 radius=0.0096
- link front_right_roller_9_link: geometry collision capsule length=0.018 radius=0.0096
Joints:
- added joint aruco_black_joint: type fixed, parent aruco_link, child aruco_black_link, origin xyz=0 0 0 rpy=0 0 0
- added joint aruco_joint: type fixed, parent support_link, child aruco_link, origin xyz=-0.075 0.0162 0.0867 rpy=-1.15192 0 0
- added joint lidar_a1_frame_joint: type fixed, parent lidar_link, child lidar_a1_frame, origin xyz=0 0 0 rpy=0 0 3.141592653589793
- added joint ms200_joint: type fixed, parent support_link, child ms200_link, origin xyz=0.0 0.1003 -0.0657 rpy=0 1.15192 1.5708
- added joint screen_joint: type fixed, parent base_link, child screen_link, origin xyz=-0.13449 0 0.082796 rpy=0 0 1.5708
- added joint support_joint: type fixed, parent base_link, child support_link, origin xyz=-0.075 0 0.195 rpy=1.15192 0 -1.5708
- joint lidar_frame_joint: origin xyz=0 0 0 rpy=0 0 3.141592653589793 -> xyz=0.0 0.1003 -0.0657 rpy=0 1.15192 1.5708; parent lidar_link -> support_link

File: src/mi_proyecto_sim/urdf/jetauto/jetauto_sim.urdf.xacro (robot description, xacro)
@@ -17,8 +17,13 @@
 <robot name="jetauto" xmlns:xacro="http://www.ros.org/wiki/xacro">
   <xacro:arg name="prefix"     default=""/>
+  <xacro:arg name="use_aruco"  default="true"/>
+  <!-- use_soporte=true (DEFAULT): soporte 3D (Legera) + ArUco 3D + MS200 (/scan, lidar_frame) +
+       A1 secundario (/scan_a1). use_soporte=false: config original (A1 en /scan, ArUco plano). -->
+  <xacro:arg name="use_soporte" default="true"/>
   <xacro:include filename="$(find mi_proyecto_sim)/urdf/jetauto/jetauto_base.urdf.xacro"/>
   <xacro:include filename="$(find mi_proyecto_sim)/urdf/jetauto/jetauto_mecanum_wheel.urdf.xacro"/>
   <xacro:include filename="$(find mi_proyecto_sim)/urdf/jetauto/jetauto_sensors.urdf.xacro"/>
   <xacro:include filename="$(find mi_proyecto_sim)/urdf/jetauto/jetauto_control.urdf.xacro"/>
+  <xacro:include filename="$(find mi_proyecto_sim)/urdf/jetauto/jetauto_soporte.urdf.xacro"/>
   <!-- chassis + decorative shells -->
   <xacro:jetauto_base prefix="$(arg prefix)"/>
@@ -32,5 +37,40 @@
   <!-- velocity ros2_control + ign_ros2_control -->
   <xacro:jetauto_control prefix="$(arg prefix)"/>
-  <!-- (Marcador ArUco del techo eliminado: lo usaba el dron para localizar el
-       carrito; no se usa en las tareas de KF + mapa de ocupacion.) -->
+  <!-- ArUco PLANO en el techo (config original). Solo cuando NO se usa el soporte 3D;
+       con use_soporte:=true lo reemplaza el ArUco 3D del jetauto_soporte. -->
+  <xacro:if value="$(arg use_aruco)">
+    <link name="techo_aruco_link">
+      <visual>
+        <geometry><box size="0.18 0.18 0.001"/></geometry>
+      </visual>
+      <collision>
+        <geometry><box size="0.18 0.18 0.001"/></geometry>
+      </collision>
+      <inertial>
+        <mass value="0.05"/>
+        <inertia ixx="0.0005" ixy="0" ixz="0" iyy="0.0005" iyz="0" izz="0.0005"/>
+      </inertial>
+    </link>
+    <gazebo reference="techo_aruco_link">
+      <visual>
+        <material>
+          <diffuse>1 1 1 1</diffuse>
+          <pbr>
+            <metal>
+              <albedo_map>file://$(find mi_proyecto_sim)/models/marcador_aruco/materials/textures/aruco4.png</albedo_map>
+            </metal>
+          </pbr>
+        </material>
+      </visual>
+    </gazebo>
+    <joint name="aruco_base_joint" type="fixed">
+      <parent link="base_link"/>
+      <child  link="techo_aruco_link"/>
+      <origin xyz="0 0 0.22" rpy="0 0 0"/>
+    </joint>
+  </xacro:if>
+  <!-- Soporte 3D (Legera) + ArUco 3D (ID 4) + MS200 funcional sobre el soporte. -->
+  <xacro:if value="$(arg use_soporte)">
+    <xacro:jetauto_soporte prefix="$(arg prefix)"/>
+  </xacro:if>
 </robot>
